Commit message: added camera_cable_frame

File: gtsp_trajectory/ur20_description/ur20_with_camera.urdf (robot description, URDF)
Before this commit: robot ur, 17 links, 16 joints
Links:
- added link camera_cable_frame; collision box size=0.06 0.1 0.06; visual box size=0.06 0.1 0.06
- link base_link_inertia: geometry collision mesh filename=package://ur_description/meshes/ur20/collision/base.stl; visual mesh filename=package://ur_description/meshes/ur20/visual/base.dae
- link camera_link: geometry collision mesh filename=package://ur_description/meshes/camera/camera.stl scale=1.0 1.0 1.0; visual mesh filename=package://ur_description/meshes/camera/camera.stl scale=1.0 1.0 1.0
- link forearm_link: geometry collision mesh filename=package://ur_description/meshes/ur20/collision/forearm.stl; visual mesh filename=package://ur_description/meshes/ur20/visual/forearm.dae
- link shoulder_link: geometry collision mesh filename=package://ur_description/meshes/ur20/collision/shoulder.stl; visual mesh filename=package://ur_description/meshes/ur20/visual/shoulder.dae
- link upper_arm_link: geometry collision mesh filename=package://ur_description/meshes/ur20/collision/upperarm.stl; visual mesh filename=package://ur_description/meshes/ur20/visual/upperarm.dae
- link wrist_1_link: geometry collision mesh filename=package://ur_description/meshes/ur20/collision/wrist1.stl; visual mesh filename=package://ur_description/meshes/ur20/visual/wrist1.dae
- link wrist_2_link: geometry collision mesh filename=package://ur_description/meshes/ur20/collision/wrist2.stl; visual mesh filename=package://ur_description/meshes/ur20/visual/wrist2.dae
- link wrist_3_link: geometry collision mesh filename=package://ur_description/meshes/ur20/collision/wrist3.stl; visual mesh filename=package://ur_description/meshes/ur20/visual/wrist3.dae
Joints:
- added joint camera_cable_frame_joint: type fixed, parent tool0, child camera_cable_frame, origin xyz=0 -0.1 -0.03 rpy=0 0 0

File: robot_ws/src/ur/Universal_Robots_ROS2_Description/urdf/ur20_with_camera.urdf (robot description, URDF)
Before this commit: robot ur, 17 links, 16 joints
Links:
- added link camera_cable_frame; collision box size=0.06 0.1 0.06; visual box size=0.06 0.1 0.06
Joints:
- added joint camera_cable_frame_joint: type fixed, parent tool0, child camera_cable_frame, origin xyz=0 -0.1 -0.03 rpy=0 0 0

File: robot_ws/src/ur/Universal_Robots_ROS2_Description/urdf/ur20_with_camera.urdf.xacro (robot description, xacro)
@@ -86,4 +86,26 @@
      <origin xyz="0 0 0" rpy="0 0 0"/>
   </xacro:ur_robot>
+  <joint name="camera_cable_frame_joint" type="fixed">
+    <origin rpy="0 0 0" xyz="0 -0.1 -0.03"/>
+    <parent link="tool0"/>
+    <child link="camera_cable_frame"/>
+  </joint>
+  <link name="camera_cable_frame">
+    <visual>
+      <origin xyz="0 0 0" rpy="0 0 0"/>
+      <geometry>
+        <box size="0.06 0.1 0.06"/>
+      </geometry>
+      <material name="dark_grey">
+        <color rgba="0.2 0.2 0.2 1.0"/>
+      </material>
+    </visual>
+    <collision>
+      <origin xyz="0 0 0" rpy="0 0 0"/>
+      <geometry>
+        <box size="0.06 0.1 0.06"/>
+      </geometry>
+    </collision>
+  </link>
   <joint name="camera_frame_1_joint" type="fixed">
     <origin rpy="0 0 0" xyz="0 0 0.0055"/>

File: robot_ws/src/ur/Universal_Robots_ROS2_Driver/ur_moveit_config/srdf/ur_with_camera_macro.srdf.xacro (robot description, xacro)
@@ -45,4 +45,9 @@
     <disable_collisions link1="${prefix}base_link" link2="${prefix}base_link_inertia" reason="Adjacent" />
     <disable_collisions link1="${prefix}base_link_inertia" link2="${prefix}shoulder_link" reason="Adjacent" />
+    <disable_collisions link1="camera_cable_frame" link2="${prefix}wrist_3_link" reason="Never" />
+    <disable_collisions link1="camera_cable_frame" link2="${prefix}tool0" reason="Adjacent" />
+    <disable_collisions link1="camera_cable_frame" link2="camera_frame_1" reason="Never" />
+    <disable_collisions link1="camera_cable_frame" link2="camera_frame_2" reason="Never" />
+    <disable_collisions link1="camera_cable_frame" link2="camera_link" reason="Never" />
     <disable_collisions link1="camera_frame_1" link2="${prefix}wrist_1_link" reason="Never" />
     <disable_collisions link1="camera_frame_1" link2="${prefix}wrist_2_link" reason="Never" />
